File: f042-3fet.kicad_pcb (KiCad board)
At the start: 2 copper layers, 42.5 x 29 mm, 39 parts, among them P1 CONN_01X02, P2 CONN_01X02, P3 CONN_01X03, Q1 Q_NMOS_GDSD, Q2 Q_NMOS_GDSD, Q3 Q_NMOS_GDSD, U1 china-switcher, U2 MCP1754ST-3302E/MB, U3 STM32F042K6Tx, U4 TJA1051T/3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

Commit message: first production
Routing:
- net /STM32F0x2-LQFP32/SWCLK: track 7.28 -> 6.16 mm
- net OUT0_UC: track 16.4 -> 17.1 mm
- net GND: track 24.6 -> 24.0 mm
Other:
- rule pad_to_mask_clearance: 0.2 -> 0.05
